Commit message: test

File: src/simple_arm/description/markII.3.urdf (robot description, URDF)
Before this commit: robot MarkII_urdf, 9 links, 8 joints
Links:
- link base_link: geometry collision mesh filename=meshes/base_link.stl scale=0.001 0.001 0.001; visual mesh filename=meshes/base_link.stl scale=0.001 0.001 0.001
- link link1: geometry collision mesh filename=meshes/link1.stl scale=0.001 0.001 0.001; visual mesh filename=meshes/link1.stl scale=0.001 0.001 0.001
- link link2: geometry collision mesh filename=meshes/link2.stl scale=0.001 0.001 0.001; visual mesh filename=meshes/link2.stl scale=0.001 0.001 0.001
- link link3: geometry collision mesh filename=meshes/link3.stl scale=0.001 0.001 0.001; visual mesh filename=meshes/link3.stl scale=0.001 0.001 0.001
- link link4: geometry collision mesh filename=meshes/link4.stl scale=0.001 0.001 0.001; visual mesh filename=meshes/link4.stl scale=0.001 0.001 0.001
- link link5: geometry collision mesh filename=meshes/link5.stl scale=0.001 0.001 0.001; visual mesh filename=meshes/link5.stl scale=0.001 0.001 0.001
- link link6: geometry collision mesh filename=meshes/link6.stl scale=0.001 0.001 0.001; visual mesh filename=meshes/link6.stl scale=0.001 0.001 0.001
- link link7: geometry collision mesh filename=meshes/link7.stl scale=0.001 0.001 0.001; visual mesh filename=meshes/link7.stl scale=0.001 0.001 0.001
- link link8: geometry collision mesh filename=meshes/link8.stl scale=0.001 0.001 0.001; visual mesh filename=meshes/link8.stl scale=0.001 0.001 0.001
Joints:
- removed joint link7_Slider-9
- added joint link6_Slider-9: type prismatic, parent link6, child link8, origin xyz=0.015700000000000058 -0.034000140000000005 0.03283129000000003 rpy=-1.5707963267948966 1.0471975511965943 -1.5707963267949128, axis -6.540341824007072e-15 -7.88860905221017e-31 0.9999999999999999, limit lower=0.0 upper=0.045 effort=1000000 velocity=1000000
- joint link1_Revolute-3: axis -1 -9.86076131526265e-32 -2.91433543964095e-15 -> 0.9999999999999999 -9.86076131526265e-32 -2.91433543964095e-15
- joint link3_Revolute-5: axis 0.0 1.0 -3.6755994903979264e-17 -> 0.0 -1.0 -3.6755994903979264e-17
- joint link5_Revolute-7: axis 0.0 1.0 -4.3859902218644406e-16 -> 0.0 -1.0 -4.3859902218644406e-16
