Commit message: changes

File: src/simple_arm/description/MarkII_urdf.urdf (robot description, URDF)
Before this commit: robot MarkII_urdf, 9 links, 8 joints
Joints:
- joint link1_Revolute-3: limit lower=-0.349066 upper=3.490659 effort=1000000 velocity=1000000 -> lower=-0.349066 upper=3.490659 effort=1000000.0 velocity=1000000.0
- joint link2_Revolute-4: limit lower=0.0 upper=3.403392 effort=1000000 velocity=1000000 -> lower=0.0 upper=3.403392 effort=1000000.0 velocity=1000000.0
- joint link4_Revolute-6: limit lower=-1.658063 upper=1.658063 effort=1000000 velocity=1000000 -> lower=-1.658063 upper=1.658063 effort=1000000.0 velocity=1000000.0
- joint link6_Slider-8: limit lower=0.0 upper=0.045 effort=1000000 velocity=1000000 -> lower=0.0 upper=0.045 effort=1000000.0 velocity=1000000.0
- joint link7_Slider-9: limit lower=0.045 upper=0.0 effort=1000000 velocity=1000000 -> lower=0.045 upper=0.0 effort=1000000.0 velocity=1000000.0
